File: circuit/_autosave-quadcopter.kicad_sch (KiCad schematic)
At the start: 100 parts, among them J1 Conn_01x01_Female, J10 Conn_01x01_Female, J11 Conn_01x01_Female, J12 Conn_01x01_Female, J13 Conn_01x01_Female, J15 Conn_01x01_Female, J18 USB_C_Receptacle_USB2.0, J19 Conn_01x08_Male, J2 Conn_01x01_Female, J20 Conn_01x04_Male, J21 Conn_01x01_Female, J22 Conn_01x01_Female, J23 Conn_01x01_Female, J24 Conn_01x01_Female, J25 Conn_01x01_Female, J26 Conn_01x01_Female, J27 Conn_01x01_Female, J28 Conn_01x01_Female, J29 Conn_01x01_Female, J3 Conn_01x01_Female, J30 Conn_01x01_Female, J31 Conn_01x01_Female, J32 Conn_01x01_Female, J33 Conn_01x01_Female, J34 Conn_01x01_Female, J36 Conn_01x01_Female, J37 Conn_01x01_Female, J38 Conn_01x01_Female, J39 Conn_01x01_Female, J4 Conn_01x01_Female, J40 Conn_01x01_Female, J41 Conn_01x01_Female, J42 Conn_01x01_Female, J43 Conn_01x01_Female, J44 Conn_01x01_Female, J45 Conn_01x01_Female, J46 Conn_01x01_Female, J47 Conn_01x01_Female, J48 Conn_01x01_Female, J49 Conn_01x01_Female, J5 Conn_01x01_Female, J50 Conn_01x01_Female, J6 Conn_01x01_Female, J7 Conn_01x01_Female, J8 Conn_01x01_Female, J9 Conn_01x01_Female, SW1 SW_DIP_x01, U1 STM32G431CBU6, U2 ICM-42605, U3 DPS310, U4 3V3, U5 5V, U6 AT7456E, U7 W25Q128JVS, Y1 16M, Y2 27M

Commit message: Added alt hold autopilot mode to Acro
Parts:
- removed J5, J6: Conn_01x01_Female, TestPoint:TestPoint_Pad_2.0x2.0mm, symbol Connector:Conn_01x01_Female
Connections:
- net SCL1: now also U1.36 (PA13)
- net SDA1: now also U1.37 (PA14)
Other:
- note added: "10v reg for cam and vtx?"
- note added: "Provide both 5v and 3v3 for UART, to accomodate various devices"
- moved on the sheet: J31, J47
Changed lines of the file:
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@@
     (effects (font (size 1.27 1.27)) (justify right bottom))
   )
+  (text "10v reg for cam and vtx?" (at 275.59 191.77 0)
+    (effects (font (size 1.27 1.27)) (justify left bottom))
+  )
+  (text "Provide both 5v and \n3v3 for UART, to accomodate various\ndevices"
+    (at 360.68 157.48 0)
+    (effects (font (size 1.27 1.27)) (justify left bottom))
+  )
   (text "ESC (iflight-layout header)" (at 355.6 22.86 180)
     (effects (font (size 1.27 1.27)) (justify right bottom))
@@
     (effects (font (size 1.27 1.27)) (justify left bottom))
   )
+  (label "SDA1" (at 113.03 114.3 180)
+    (effects (font (size 1.27 1.27)) (justify right bottom))
+  )
   (label "M3_PWM" (at 377.19 35.56 180)
     (effects (font (size 1.27 1.27)) (justify right bottom))
@@
     (effects (font (size 1.27 1.27)) (justify right bottom))
   )
-  (label "SCL3" (at 325.12 193.04 180)
-    (effects (font (size 1.27 1.27)) (justify right bottom))
-  )
   (label "NRST" (at 34.29 35.56 180)
     (effects (font (size 1.27 1.27)) (justify right bottom))
@@
     (effects (font (size 1.27 1.27)) (justify left bottom))
   )
-  (label "SDA3" (at 325.12 198.12 180)
-    (effects (font (size 1.27 1.27)) (justify right bottom))
-  )
   (label "USB_N" (at 64.77 205.74 0)
     (effects (font (size 1.27 1.27)) (justify left bottom))
@@
     (effects (font (size 1.27 1.27)) (justify right bottom))
   )
+  (label "SCL1" (at 113.03 111.76 180)
+    (effects (font (size 1.27 1.27)) (justify right bottom))
+  )
   (label "M1_PWM" (at 342.9 50.8 180)
     (effects (font (size 1.27 1.27)) (justify right bottom))
@@
     (pin "1")
   )
-  (symbol (lib_id "power:+5V") (at 325.12 163.83 90) (unit 1)
+  (symbol (lib_id "power:+5V") (at 374.65 158.75 90) (unit 1)
     (in_bom yes) (on_board yes) (fields_autoplaced)
-    (property "Reference" "#PWR0144" (id 0) (at 328.93 163.83 0)
+    (property "Reference" "#PWR0144" (id 0) (at 378.46 158.75 0)
       (effects (font (size 1.27 1.27)) hide)
     )
-    (property "Value" "+5V" (id 1) (at 321.31 163.8299 90)
+    (property "Value" "+5V" (id 1) (at 370.84 158.7499 90)
       (effects (font (size 1.27 1.27)) (justify left))
     )
-    (property "Footprint" "" (id 2) (at 325.12 163.83 0)
+    (property "Footprint" "" (id 2) (at 374.65 158.75 0)
       (effects (font (size 1.27 1.27)) hide)
     )
-    (property "Datasheet" "" (id 3) (at 325.12 163.83 0)
+    (property "Datasheet" "" (id 3) (at 374.65 158.75 0)
       (effects (font (size 1.27 1.27)) hide)
     )
@@
     (pin "2")
   )
-  (symbol (lib_id "Connector:Conn_01x01_Female") (at 330.2 198.12 0) (unit 1)
-    (in_bom yes) (on_board yes) (fields_autoplaced)
-    (property "Reference" "J6" (id 0) (at 331.47 196.8499 0)
-      (effects (font (size 1.27 1.27)) (justify left))
-    )
-    (property "Value" "Conn_01x01_Female" (id 1) (at 331.47 199.3899 0)
-      (effects (font (size 1.27 1.27)) (justify left))
-    )
-    (property "Footprint" "TestPoint:TestPoint_Pad_2.0x2.0mm" (id 2) (at 330.2 198.12 0)
-      (effects (font (size 1.27 1.27)) hide)
-    )
-    (property "Datasheet" "~" (id 3) (at 330.2 198.12 0)
-      (effects (font (size 1.27 1.27)) hide)
-    )
-    (pin "1")
-  )
   (symbol (lib_id "Connector:Conn_01x01_Female") (at 381 242.57 0) (unit 1)
     (in_bom yes) (on_board yes) (fields_autoplaced)
@@
     (pin "9")
   )
-  (symbol (lib_id "power:GND") (at 325.12 168.91 270) (unit 1)
+  (symbol (lib_id "power:GND") (at 374.65 173.99 270) (unit 1)
     (in_bom yes) (on_board yes) (fields_autoplaced)
-    (property "Reference" "#PWR0139" (id 0) (at 318.77 168.91 0)
+    (property "Reference" "#PWR0139" (id 0) (at 368.3 173.99 0)
       (effects (font (size 1.27 1.27)) hide)
     )
-    (property "Value" "GND" (id 1) (at 321.31 168.9099 90)
+    (property "Value" "GND" (id 1) (at 370.84 173.9899 90)
       (effects (font (size 1.27 1.27)) (justify right))
     )
-    (property "Footprint" "" (id 2) (at 325.12 168.91 0)
+    (property "Footprint" "" (id 2) (at 374.65 173.99 0)
       (effects (font (size 1.27 1.27)) hide)
     )
-    (property "Datasheet" "" (id 3) (at 325.12 168.91 0)
+    (property "Datasheet" "" (id 3) (at 374.65 173.99 0)
       (effects (font (size 1.27 1.27)) hide)
     )
     (pin "1")
   )
-  (symbol (lib_id "Connector:Conn_01x01_Female") (at 330.2 163.83 0) (unit 1)
+  (symbol (lib_id "Connector:Conn_01x01_Female") (at 379.73 158.75 0) (unit 1)
     (in_bom yes) (on_board yes) (fields_autoplaced)
-    (property "Reference" "J47" (id 0) (at 331.47 162.5599 0)
+    (property "Reference" "J47" (id 0) (at 381 157.4799 0)
       (effects (font (size 1.27 1.27)) (justify left))
     )
-    (property "Value" "Conn_01x01_Female" (id 1) (at 331.47 165.0999 0)
+    (property "Value" "Conn_01x01_Female" (id 1) (at 381 160.0199 0)
       (effects (font (size 1.27 1.27)) (justify left))
     )
-    (property "Footprint" "TestPoint:TestPoint_Pad_2.0x2.0mm" (id 2) (at 330.2 163.83 0)
+    (property "Footprint" "TestPoint:TestPoint_Pad_2.0x2.0mm" (id 2) (at 379.73 158.75 0)
       (effects (font (size 1.27 1.27)) hide)
     )
-    (property "Datasheet" "~" (id 3) (at 330.2 163.83 0)
+    (property "Datasheet" "~" (id 3) (at 379.73 158.75 0)
       (effects (font (size 1.27 1.27)) hide)
     )
@@
     (pin "1")
   )
-  (symbol (lib_id "Connector:Conn_01x01_Female") (at 330.2 168.91 0) (unit 1)
+  (symbol (lib_id "Connector:Conn_01x01_Female") (at 379.73 173.99 0) (unit 1)
     (in_bom yes) (on_board yes) (fields_autoplaced)
-    (property "Reference" "J31" (id 0) (at 331.47 167.6399 0)
+    (property "Reference" "J31" (id 0) (at 381 172.7199 0)
       (effects (font (size 1.27 1.27)) (justify left))
     )
-    (property "Value" "Conn_01x01_Female" (id 1) (at 331.47 170.1799 0)
+    (property "Value" "Conn_01x01_Female" (id 1) (at 381 175.2599 0)
       (effects (font (size 1.27 1.27)) (justify left))
     )
-    (property "Footprint" "TestPoint:TestPoint_Pad_2.0x2.0mm" (id 2) (at 330.2 168.91 0)
+    (property "Footprint" "TestPoint:TestPoint_Pad_2.0x2.0mm" (id 2) (at 379.73 173.99 0)
       (effects (font (size 1.27 1.27)) hide)
     )
-    (property "Datasheet" "~" (id 3) (at 330.2 168.91 0)
+    (property "Datasheet" "~" (id 3) (at 379.73 173.99 0)
       (effects (font (size 1.27 1.27)) hide)
     )
@@
     (pin "1")
   )
-  (symbol (lib_id "Connector:Conn_01x01_Female") (at 330.2 193.04 0) (unit 1)
-    (in_bom yes) (on_board yes) (fields_autoplaced)
-    (property "Reference" "J5" (id 0) (at 331.47 191.7699 0)
-      (effects (font (size 1.27 1.27)) (justify left))
-    )
-    (property "Value" "Conn_01x01_Female" (id 1) (at 331.47 194.3099 0)
-      (effects (font (size 1.27 1.27)) (justify left))
-    )
-    (property "Footprint" "TestPoint:TestPoint_Pad_2.0x2.0mm" (id 2) (at 330.2 193.04 0)
-      (effects (font (size 1.27 1.27)) hide)
-    )
-    (property "Datasheet" "~" (id 3) (at 330.2 193.04 0)
-      (effects (font (size 1.27 1.27)) hide)
-    )
-    (pin "1")
-  )
   (symbol (lib_id "Device:R") (at 60.96 205.74 90) (unit 1)
     (in_bom yes) (on_board yes)
@@
       (reference "J4") (unit 1) (value "Conn_01x01_Female") (footprint "TestPoint:TestPoint_Pad_1.0x1.0mm")
     )
-    (path "/f07b7011-426d-4eed-b616-bff89b8b3959"
-      (reference "J5") (unit 1) (value "Conn_01x01_Female") (footprint "TestPoint:TestPoint_Pad_2.0x2.0mm")
-    )
-    (path "/31cc448a-552a-428f-858d-5e1ebc618542"
-      (reference "J6") (unit 1) (value "Conn_01x01_Female") (footprint "TestPoint:TestPoint_Pad_2.0x2.0mm")
-    )
     (path "/e491e9c4-83e3-4bb2-8ba8-b05d76f48b2c"
