File: circuit/_autosave-quadcopter.kicad_sch (KiCad schematic)
At the start: 115 parts, among them J1 Conn_01x01_Female, J10 Conn_01x01_Female, J12 Conn_01x01_Female, J13 Conn_01x01_Female, J15 Conn_01x01_Female, J16 Conn_01x01_Female, J17 Conn_01x01_Female, J18 USB_C_Receptacle_USB2.0, J19 Conn_01x08_Male, J2 Conn_01x01_Female, J21 Conn_01x01_Female, J22 Conn_01x01_Female, J23 Conn_01x01_Female, J24 Conn_01x01_Female, J25 Conn_01x01_Female, J26 Conn_01x01_Female, J28 Conn_01x01_Female, J29 Conn_01x01_Female, J3 Conn_01x01_Female, J30 Conn_01x01_Female, J31 Conn_01x01_Female, J32 Conn_01x01_Female, J33 Conn_01x01_Female, J34 Conn_01x01_Female, J36 Conn_01x01_Female, J37 Conn_01x01_Female, J38 Conn_01x01_Female, J39 Conn_01x01_Female, J4 Conn_01x01_Female, J40 Conn_01x01_Female, J41 Conn_01x01_Female, J42 Conn_01x01_Female, J43 Conn_01x01_Female, J44 Conn_01x01_Female, J45 Conn_01x01_Female, J46 Conn_01x01_Female, J47 Conn_01x01_Female, J48 Conn_01x01_Female, J49 Conn_01x01_Female, J50 Conn_01x01_Female, J6 Conn_01x04_Male, J7 Conn_01x01_Female, J8 Conn_01x01_Female, J9 Conn_01x01_Female, SW1 SW_DIP_x01, U1 STM32G431CBU6, U2 ICM-42605, U3 DPS310, U4 3V3, U5 5V, U6 AT7456E, U7 W25Q128JVS, U8 SX1281, Y1 16M, Y2 27M

Commit message: Lots of work on board, including removing RSSI
Parts:
- removed AE1: Antenna, Connector_Coaxial:U.FL_Molex_MCRF_73412-0110_Vertical, symbol Device:Antenna
- removed J3, J4: Conn_01x01_Female, TestPoint:TestPoint_Pad_1.0x1.0mm, symbol Connector:Conn_01x01_Female
- added J5: Conn_Coaxial, Connector_Coaxial:U.FL_Hirose_U.FL-R-SMT-1_Vertical, symbol Connector:Conn_Coaxial
- J6: value Conn_01x04_Male -> Conn_01x06_Male; footprint Connector_JST:JST_SH_BM04B-SRSS-TB_1x04-1MP_P1.00mm_Vertical -> Connector_JST:JST_SH_BM06B-SRSS-TB_1x06-1MP_P1.00mm_Vertical; symbol Connector:Conn_01x04_Male -> Connector:Conn_01x06_Male
Connections:
- net +5V: now also J6.5 (Pin_5)
- net GND: now also J6.4 (Pin_4), J5.2 (Ext)
- net VID_IN: now also J6.6 (Pin_6)
- net at U8.22 (RFIO): now also J5.1 (In)
Other:
- moved on the sheet: J28, J29

Commit message: more routing
Other:
- moved on the sheet: J5, R16, R18
Changed lines of the file:
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@@
   (junction (at 100.33 76.2) (diameter 0) (color 0 0 0 0)
   )
-  (junction (at 58.42 140.97) (diameter 0) (color 0 0 0 0)
+  (junction (at 58.42 130.81) (diameter 0) (color 0 0 0 0)
   )
   (junction (at 189.23 68.58) (diameter 0) (color 0 0 0 0)
@@
     (stroke (width 0) (type default) (color 0 0 0 0))
   )
-  (wire (pts (xy 58.42 140.97) (xy 58.42 147.32))
+  (wire (pts (xy 58.42 130.81) (xy 58.42 137.16))
     (stroke (width 0) (type default) (color 0 0 0 0))
   )
@@
     (stroke (width 0) (type default) (color 0 0 0 0))
   )
-  (wire (pts (xy 55.88 140.97) (xy 58.42 140.97))
+  (wire (pts (xy 55.88 130.81) (xy 58.42 130.81))
     (stroke (width 0) (type default) (color 0 0 0 0))
   )
@@
     (stroke (width 0) (type default) (color 0 0 0 0))
   )
-  (wire (pts (xy 78.74 311.15) (xy 88.9 311.15))
-    (stroke (width 0) (type default) (color 0 0 0 0))
-  )
   (wire (pts (xy 85.09 72.39) (xy 95.25 72.39))
     (stroke (width 0) (type default) (color 0 0 0 0))
@@
     (stroke (width 0) (type default) (color 0 0 0 0))
   )
-  (wire (pts (xy 58.42 140.97) (xy 60.96 140.97))
+  (wire (pts (xy 58.42 130.81) (xy 60.96 130.81))
     (stroke (width 0) (type default) (color 0 0 0 0))
   )
@@
     (stroke (width 0) (type default) (color 0 0 0 0))
   )
-  (text "todo: What resistor vls for cur?" (at 50.8 133.35 0)
+  (text "todo: What resistor vls for cur?" (at 50.8 123.19 0)
     (effects (font (size 1.27 1.27)) (justify left bottom))
   )
@@
     (effects (font (size 1.27 1.27)) (justify right bottom))
   )
-  (label "CURRENT" (at 165.1 96.52 0)
-    (effects (font (size 1.27 1.27)) (justify left bottom))
-  )
   (label "CUR_DIV" (at 165.1 99.06 0)
     (effects (font (size 1.27 1.27)) (justify left bottom))
@@
     (effects (font (size 1.27 1.27)) (justify right bottom))
   )
-  (label "CURRENT" (at 48.26 140.97 180)
+  (label "CURRENT" (at 48.26 130.81 180)
     (effects (font (size 1.27 1.27)) (justify right bottom))
   )
@@
     (effects (font (size 1.27 1.27)) (justify left bottom))
   )
-  (label "CUR_DIV" (at 58.42 147.32 0)
+  (label "CUR_DIV" (at 58.42 137.16 0)
     (effects (font (size 1.27 1.27)) (justify left bottom))
   )
@@
     (pin "2")
   )
-  (symbol (lib_id "power:GND") (at 68.58 140.97 90) (unit 1)
+  (symbol (lib_id "power:GND") (at 68.58 130.81 90) (unit 1)
     (in_bom yes) (on_board yes)
-    (property "Reference" "#PWR0171" (id 0) (at 74.93 140.97 0)
+    (property "Reference" "#PWR0171" (id 0) (at 74.93 130.81 0)
       (effects (font (size 1.27 1.27)) hide)
     )
-    (property "Value" "GND" (id 1) (at 71.8312 140.843 90)
+    (property "Value" "GND" (id 1) (at 71.8312 130.683 90)
       (effects (font (size 1.27 1.27)) (justify right))
     )
-    (property "Footprint" "" (id 2) (at 68.58 140.97 0)
+    (property "Footprint" "" (id 2) (at 68.58 130.81 0)
       (effects (font (size 1.27 1.27)) hide)
     )
-    (property "Datasheet" "" (id 3) (at 68.58 140.97 0)
+    (property "Datasheet" "" (id 3) (at 68.58 130.81 0)
       (effects (font (size 1.27 1.27)) hide)
     )
@@
     (pin "1")
   )
-  (symbol (lib_id "Connector:Conn_Coaxial") (at 93.98 311.15 0) (unit 1)
+  (symbol (lib_id "Connector:Conn_Coaxial") (at 83.82 311.15 0) (unit 1)
     (in_bom yes) (on_board yes) (fields_autoplaced)
-    (property "Reference" "J5" (id 0) (at 96.52 310.1731 0)
+    (property "Reference" "J5" (id 0) (at 86.36 310.1731 0)
       (effects (font (size 1.27 1.27)) (justify left))
     )
-    (property "Value" "Conn_Coaxial" (id 1) (at 96.52 312.7131 0)
+    (property "Value" "Conn_Coaxial" (id 1) (at 86.36 312.7131 0)
       (effects (font (size 1.27 1.27)) (justify left))
     )
-    (property "Footprint" "Connector_Coaxial:U.FL_Hirose_U.FL-R-SMT-1_Vertical" (id 2) (at 93.98 311.15 0)
+    (property "Footprint" "Connector_Coaxial:U.FL_Hirose_U.FL-R-SMT-1_Vertical" (id 2) (at 83.82 311.15 0)
       (effects (font (size 1.27 1.27)) hide)
     )
-    (property "Datasheet" " ~" (id 3) (at 93.98 311.15 0)
+    (property "Datasheet" " ~" (id 3) (at 83.82 311.15 0)
       (effects (font (size 1.27 1.27)) hide)
     )
-    (property "LCSC" "C88374" (id 4) (at 93.98 311.15 0)
+    (property "LCSC" "C88374" (id 4) (at 83.82 311.15 0)
       (effects (font (size 1.27 1.27)) hide)
     )
-    (property "Part" "Hirose U.FL-R-SMT-1(80)" (id 5) (at 93.98 311.15 0)
+    (property "Part" "Hirose U.FL-R-SMT-1(80)" (id 5) (at 83.82 311.15 0)
       (effects (font (size 1.27 1.27)) hide)
     )
@@
     (pin "1")
   )
-  (symbol (lib_id "Device:R") (at 64.77 140.97 270) (unit 1)
+  (symbol (lib_id "Device:R") (at 64.77 130.81 270) (unit 1)
     (in_bom yes) (on_board yes)
-    (property "Reference" "R18" (id 0) (at 64.77 138.43 90))
-    (property "Value" "1.5k" (id 1) (at 72.39 138.43 90))
-    (property "Footprint" "Resistor_SMD:R_0402_1005Metric" (id 2) (at 64.77 139.192 90)
+    (property "Reference" "R18" (id 0) (at 64.77 128.27 90))
+    (property "Value" "1.5k" (id 1) (at 72.39 128.27 90))
+    (property "Footprint" "Resistor_SMD:R_0402_1005Metric" (id 2) (at 64.77 129.032 90)
       (effects (font (size 1.27 1.27)) hide)
     )
-    (property "Datasheet" "~" (id 3) (at 64.77 140.97 0)
+    (property "Datasheet" "~" (id 3) (at 64.77 130.81 0)
       (effects (font (size 1.27 1.27)) hide)
     )
-    (property "LCSC" "C25867" (id 4) (at 64.77 140.97 0)
+    (property "LCSC" "C25867" (id 4) (at 64.77 130.81 0)
       (effects (font (size 1.27 1.27)) hide)
     )
@@
     (pin "1")
   )
-  (symbol (lib_id "Device:R") (at 52.07 140.97 270) (unit 1)
+  (symbol (lib_id "Device:R") (at 52.07 130.81 270) (unit 1)
     (in_bom yes) (on_board yes)
-    (property "Reference" "R16" (id 0) (at 46.99 137.16 90))
-    (property "Value" "10k" (id 1) (at 55.88 138.43 90))
-    (property "Footprint" "Resistor_SMD:R_0402_1005Metric" (id 2) (at 52.07 139.192 90)
+    (property "Reference" "R16" (id 0) (at 46.99 127 90))
+    (property "Value" "10k" (id 1) (at 55.88 128.27 90))
+    (property "Footprint" "Resistor_SMD:R_0402_1005Metric" (id 2) (at 52.07 129.032 90)
       (effects (font (size 1.27 1.27)) hide)
     )
-    (property "Datasheet" "~" (id 3) (at 52.07 140.97 0)
+    (property "Datasheet" "~" (id 3) (at 52.07 130.81 0)
       (effects (font (size 1.27 1.27)) hide)
     )
-    (property "LCSC" "C25744" (id 4) (at 52.07 140.97 0)
+    (property "LCSC" "C25744" (id 4) (at 52.07 130.81 0)
       (effects (font (size 1.27 1.27)) hide)
     )
@@
     (pin "1")
   )
-  (symbol (lib_id "power:GND") (at 93.98 316.23 0) (unit 1)
+  (symbol (lib_id "power:GND") (at 83.82 316.23 0) (unit 1)
     (in_bom yes) (on_board yes) (fields_autoplaced)
-    (property "Reference" "#PWR0165" (id 0) (at 93.98 322.58 0)
+    (property "Reference" "#PWR0165" (id 0) (at 83.82 322.58 0)
       (effects (font (size 1.27 1.27)) hide)
     )
-    (property "Value" "GND" (id 1) (at 96.52 317.4999 0)
+    (property "Value" "GND" (id 1) (at 86.36 317.4999 0)
       (effects (font (size 1.27 1.27)) (justify left))
     )
-    (property "Footprint" "" (id 2) (at 93.98 316.23 0)
+    (property "Footprint" "" (id 2) (at 83.82 316.23 0)
       (effects (font (size 1.27 1.27)) hide)
     )
-    (property "Datasheet" "" (id 3) (at 93.98 316.23 0)
+    (property "Datasheet" "" (id 3) (at 83.82 316.23 0)
       (effects (font (size 1.27 1.27)) hide)
     )

Commit message: More work on translating ELRS
Parts:
- R13, R16: value 10k -> 15k; LCSC C25744 -> C25756
Connections:
- net +3V3: no longer U8.3 (NRESET)
- new net ELRS_RST: U8.3 (NRESET)
Other:
- note added: "Voltage divider. This keeps a 8S cell at full charge (33.6v) below 3.3v"
- note added: "todo: change these to support 33.6v, for 8S."
- note removed: "Voltage divider. This keeps a 6S cell at full charge (25.2v) below 3.3v"
Changed lines of the file:
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@@
     (effects (font (size 1.27 1.27)) (justify right bottom))
   )
-  (text "Voltage divider. This keeps a 6S cell\nat full charge (25.2v) below 3.3v"
+  (text "Voltage divider. This keeps a 8S cell\nat full charge (33.6v) below 3.3v"
     (at 44.45 102.87 0)
     (effects (font (size 1.27 1.27)) (justify left bottom))
@@
     (effects (font (size 1.27 1.27)) (justify left bottom))
   )
+  (text "todo: change these to support 33.6v, for 8S." (at 35.56 119.38 0)
+    (effects (font (size 1.27 1.27)) (justify left bottom))
+  )
   (text "Using Diatone pinout, since it's\nperhaps the most popular (2022)"
     (at 312.42 17.78 0)
@@
     (effects (font (size 1.27 1.27)) (justify left bottom))
   )
+  (label "ELRS_RST" (at 48.26 289.56 180)
+    (effects (font (size 1.27 1.27)) (justify right bottom))
+  )
   (label "SCK_3" (at 78.74 300.99 0)
     (effects (font (size 1.27 1.27)) (justify left bottom))
@@
     (effects (font (size 1.27 1.27)) (justify left bottom))
   )
+  (label "ELRS_RST" (at 165.1 101.6 180)
+    (effects (font (size 1.27 1.27)) (justify right bottom))
+  )
   (label "CS_ELRS" (at 109.22 64.77 180)
     (effects (font (size 1.27 1.27)) (justify right bottom))
@@
     (in_bom yes) (on_board yes)
     (property "Reference" "R13" (id 0) (at 46.99 106.68 90))
-    (property "Value" "10k" (id 1) (at 55.88 106.68 90))
+    (property "Value" "15k" (id 1) (at 55.88 106.68 90))
     (property "Footprint" "Resistor_SMD:R_0402_1005Metric" (id 2) (at 52.07 107.442 90)
       (effects (font (size 1.27 1.27)) hide)
@@
       (effects (font (size 1.27 1.27)) hide)
     )
-    (property "LCSC" "C25744" (id 4) (at 52.07 109.22 0)
+    (property "LCSC" "C25756" (id 4) (at 52.07 109.22 0)
       (effects (font (size 1.27 1.27)) hide)
     )
@@
     (in_bom yes) (on_board yes)
     (property "Reference" "R16" (id 0) (at 46.99 127 90))
-    (property "Value" "10k" (id 1) (at 55.88 128.27 90))
+    (property "Value" "15k" (id 1) (at 55.88 128.27 90))
     (property "Footprint" "Resistor_SMD:R_0402_1005Metric" (id 2) (at 52.07 129.032 90)
       (effects (font (size 1.27 1.27)) hide)
@@
       (effects (font (size 1.27 1.27)) hide)
     )
-    (property "LCSC" "C25744" (id 4) (at 52.07 130.81 0)
+    (property "LCSC" "C25756" (id 4) (at 52.07 130.81 0)
       (effects (font (size 1.27 1.27)) hide)
     )
@@
     (pin "2")
   )
-  (symbol (lib_id "power:+3V3") (at 48.26 289.56 90) (unit 1)
-    (in_bom yes) (on_board yes) (fields_autoplaced)
-    (property "Reference" "#PWR0175" (id 0) (at 52.07 289.56 0)
-      (effects (font (size 1.27 1.27)) hide)
-    )
-    (property "Value" "+3V3" (id 1) (at 44.45 289.5599 90)
-      (effects (font (size 1.27 1.27)) (justify left))
-    )
-    (property "Footprint" "" (id 2) (at 48.26 289.56 0)
-      (effects (font (size 1.27 1.27)) hide)
-    )
-    (property "Datasheet" "" (id 3) (at 48.26 289.56 0)
-      (effects (font (size 1.27 1.27)) hide)
-    )
-    (pin "1")
-  )
   (symbol (lib_id "power:GND") (at 193.04 91.44 270) (unit 1)
     (in_bom yes) (on_board yes) (fields_autoplaced)
@@
       (reference "#PWR0174") (unit 1) (value "+3V3") (footprint "")
     )
-    (path "/d1e82e3b-23cb-4236-bf46-66c8b8043eb5"
-      (reference "#PWR0175") (unit 1) (value "+3V3") (footprint "")
-    )
     (path "/38939625-bd2a-4876-8a30-a5626a6df1f6"
       (reference "#PWR0177") (unit 1) (value "+BATT") (footprint "")
@@
     )
     (path "/427ea469-a00c-48a4-8283-a7d9e027923d"
-      (reference "R13") (unit 1) (value "10k") (footprint "Resistor_SMD:R_0402_1005Metric")
+      (reference "R13") (unit 1) (value "15k") (footprint "Resistor_SMD:R_0402_1005Metric")
     )
     (path "/667f12d7-16dd-4278-bb5b-b991203c0138"
@@
     )
     (path "/cc86727f-894e-486d-8510-2b64f6ee41b6"
-      (reference "R16") (unit 1) (value "10k") (footprint "Resistor_SMD:R_0402_1005Metric")
+      (reference "R16") (unit 1) (value "15k") (footprint "Resistor_SMD:R_0402_1005Metric")
     )
     (path "/9f433e30-c50f-41e7-b5fb-32b34b7ca279"

Commit message: Board is now ready for order, pending review
Connections:
- net BATT_DIV: now also U1.16 (PC4); no longer U1.19 (PB2)
- net CUR_DIV: now also U1.19 (PB2)
- net ELRS_RST: now also U1.9 (PA1)
Changed lines of the file:
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@@
     (effects (font (size 1.27 1.27)) (justify right bottom))
   )
-  (label "CUR_DIV" (at 165.1 99.06 0)
+  (label "CUR_DIV" (at 143.51 66.04 0)
     (effects (font (size 1.27 1.27)) (justify left bottom))
   )
@@
     (effects (font (size 1.27 1.27)) (justify right bottom))
   )
-  (label "BATT_DIV" (at 143.51 66.04 0)
+  (label "BATT_DIV" (at 143.51 116.84 0)
     (effects (font (size 1.27 1.27)) (justify left bottom))
   )
@@
     (effects (font (size 1.27 1.27)) (justify left bottom))
   )
-  (label "ELRS_RST" (at 165.1 101.6 180)
-    (effects (font (size 1.27 1.27)) (justify right bottom))
-  )
+  (label "ELRS_RST" (at 113.03 81.28 180)
+    (effects (font (size 1.27 1.27)) (justify right bottom))
+  )
