File: circuit/quadcopter.kicad_sch (KiCad schematic)
At the start: 114 parts, among them J1 Conn_01x01_Female, J10 Conn_01x01_Female, J11 Conn_01x01_Female, J12 Conn_01x01_Female, J13 Conn_01x01_Female, J14 Conn_01x01_Female, J15 Conn_01x01_Female, J16 Conn_01x01_Female, J17 Conn_01x01_Female, J18 USB_C_Receptacle_USB2.0, J19 Conn_01x08_Male, J2 Conn_01x01_Female, J20 Conn_01x04_Male, J21 Conn_01x01_Female, J22 Conn_01x01_Female, J23 Conn_01x01_Female, J24 Conn_01x01_Female, J25 Conn_01x01_Female, J26 Conn_01x01_Female, J27 Conn_01x01_Female, J28 Conn_01x01_Female, J29 Conn_01x01_Female, J3 Conn_01x01_Female, J30 Conn_01x01_Female, J31 Conn_01x01_Female, J32 Conn_01x01_Female, J33 Conn_01x01_Female, J34 Conn_01x01_Female, J35 Conn_01x01_Female, J36 Conn_01x01_Female, J37 Conn_01x01_Female, J38 Conn_01x01_Female, J39 Conn_01x01_Female, J4 Conn_01x01_Female, J40 Conn_01x01_Female, J41 Conn_01x01_Female, J42 Conn_01x01_Female, J43 Conn_01x01_Female, J44 Conn_01x01_Female, J45 Conn_01x01_Female, J46 Conn_01x01_Female, J47 Conn_01x01_Female, J48 Conn_01x01_Female, J49 Conn_01x01_Female, J5 Conn_01x01_Female, J50 Conn_01x01_Female, J51 Conn_01x01_Female, J6 Conn_01x01_Female, J7 Conn_01x01_Female, J8 Conn_01x01_Female, J9 Conn_01x01_Female, SW1 SW_DIP_x01, U1 STM32G431CBU6, U2 ICM-42605, U3 DPS310, U4 3V3, U5 5V, U6 AT7456E, U7 W25Q128JVS, Y1 16M, Y2 27M

Commit message: Added CRSF module for radio siganls
Parts:
- removed C?: C, symbol Device:C
- removed J35: Conn_01x01_Female, TestPoint:TestPoint_Pad_1.5x1.5mm, symbol Connector:Conn_01x01_Female
- added C27: 47u, Capacitor_SMD:C_0805_2012Metric, symbol Device:C
- L2: renamed from L?; footprint (none) -> Anyleaf_Shared:SMNR4020 inductor; LCSC (none) -> C467068
- gave numbers to parts that had none: 2
Connections:
- net +BATT: now also C27.2
- net BUZZER+: now also U1.29 (PC6)
- net GND: now also C27.1
- net UART1_RX: now also U1.45 (PB7)
- net UART1_TX: now also U1.44 (PB6)
- net UART2_TX: now also U1.10 (PA2)
- net UART3_RX: now also U1.24 (PB11)
- net UART4_RX: now also U1.40 (PC11)
- net UART4_TX: now also U1.39 (PC10)
- no-connect marks 3 -> 5
Other:
- note added: "A lower cutoff for this LC lowpass is better, but that requires a larger cap and inductor, and we're low on space."
Changed lines of the file:
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@@
   (junction (at 266.7 55.88) (diameter 0) (color 0 0 0 0)
   )
+  (no_connect (at 113.03 66.04))
+  (no_connect (at 113.03 68.58))
   (no_connect (at 27.94 231.14))
   (no_connect (at 215.9 209.55))
@@
     (effects (font (size 1.27 1.27)) (justify left bottom))
   )
+  (text "A lower cutoff for this LC lowpass is\nbetter, but that requires a larger cap\nand inductor, and we're low on space."
+    (at 284.48 104.14 0)
+    (effects (font (size 1.27 1.27)) (justify left bottom))
+  )
   (text "Flash memory for \"black box\"" (at 104.14 189.23 0)
     (effects (font (size 1.27 1.27)) (justify left bottom))
@@
     (effects (font (size 1.27 1.27)) (justify left bottom))
   )
-  (label "BUZZER-" (at 318.77 177.8 180)
-    (effects (font (size 1.27 1.27)) (justify right bottom))
-  )
   (label "VID_IN" (at 232.41 199.39 0)
     (effects (font (size 1.27 1.27)) (justify left bottom))
@@
     (effects (font (size 1.27 1.27)) (justify right bottom))
   )
-  (label "BUZZER+" (at 100.33 118.11 180)
-    (effects (font (size 1.27 1.27)) (justify right bottom))
+  (label "BUZZER+" (at 143.51 114.3 0)
+    (effects (font (size 1.27 1.27)) (justify left bottom))
   )
   (label "CURRENT" (at 342.9 38.1 180)
@@
     (effects (font (size 1.27 1.27)) (justify left bottom))
   )
+  (label "UART4_RX" (at 143.51 109.22 0)
+    (effects (font (size 1.27 1.27)) (justify left bottom))
+  )
   (label "CS_OSD" (at 190.5 229.87 180)
     (effects (font (size 1.27 1.27)) (justify right bottom))
@@
     (effects (font (size 1.27 1.27)) (justify right bottom))
   )
+  (label "UART1_RX" (at 143.51 78.74 0)
+    (effects (font (size 1.27 1.27)) (justify left bottom))
+  )
   (label "MISO_2" (at 143.51 96.52 0)
     (effects (font (size 1.27 1.27)) (justify left bottom))
@@
     (effects (font (size 1.27 1.27)) (justify left bottom))
   )
+  (label "UART1_TX" (at 147.32 116.84 0)
+    (effects (font (size 1.27 1.27)) (justify left bottom))
+  )
   (label "BAT_IN" (at 289.56 85.09 180)
     (effects (font (size 1.27 1.27)) (justify right bottom))
   )
+  (label "UART4_TX" (at 143.51 111.76 0)
+    (effects (font (size 1.27 1.27)) (justify left bottom))
+  )
   (label "SDA1" (at 325.12 237.49 180)
     (effects (font (size 1.27 1.27)) (justify right bottom))
@@
     (effects (font (size 1.27 1.27)) (justify right bottom))
   )
+  (label "UART3_RX" (at 143.51 88.9 0)
+    (effects (font (size 1.27 1.27)) (justify left bottom))
+  )
   (label "UART2_TX" (at 375.92 242.57 180)
     (effects (font (size 1.27 1.27)) (justify right bottom))
@@
     (effects (font (size 1.27 1.27)) (justify right bottom))
   )
-  (label "BUZZER-" (at 100.33 123.19 180)
-    (effects (font (size 1.27 1.27)) (justify right bottom))
-  )
   (label "MOSI_2" (at 190.5 222.25 180)
     (effects (font (size 1.27 1.27)) (justify right bottom))
@@
     (effects (font (size 1.27 1.27)) (justify left bottom))
   )
+  (label "UART1_TX" (at 143.51 76.2 0)
+    (effects (font (size 1.27 1.27)) (justify left bottom))
+  )
   (label "MOSI_3" (at 130.81 207.01 0)
     (effects (font (size 1.27 1.27)) (justify left bottom))
@@
     (effects (font (size 1.27 1.27)) (justify right bottom))
   )
+  (label "UART2_TX" (at 113.03 83.82 180)
+    (effects (font (size 1.27 1.27)) (justify right bottom))
+  )
   (label "SDA2" (at 113.03 99.06 180)
     (effects (font (size 1.27 1.27)) (justify right bottom))
@@
     (pin "1")
   )
-  (symbol (lib_id "Connector:Conn_01x01_Female") (at 323.85 177.8 0) (unit 1)
-    (in_bom yes) (on_board yes) (fields_autoplaced)
-    (property "Reference" "J35" (id 0) (at 325.12 176.5299 0)
-      (effects (font (size 1.27 1.27)) (justify left))
-    )
-    (property "Value" "Conn_01x01_Female" (id 1) (at 325.12 179.0699 0)
-      (effects (font (size 1.27 1.27)) (justify left))
-    )
-    (property "Footprint" "TestPoint:TestPoint_Pad_1.5x1.5mm" (id 2) (at 323.85 177.8 0)
-      (effects (font (size 1.27 1.27)) hide)
-    )
-    (property "Datasheet" "~" (id 3) (at 323.85 177.8 0)
-      (effects (font (size 1.27 1.27)) hide)
-    )
-    (pin "1")
-  )
   (symbol (lib_id "Connector:Conn_01x01_Female") (at 382.27 92.71 0) (unit 1)
     (in_bom yes) (on_board yes)
@@
   (symbol (lib_id "power:GND") (at 304.8 92.71 0) (unit 1)
     (in_bom yes) (on_board yes)
-    (property "Reference" "#PWR?" (id 0) (at 304.8 99.06 0)
+    (property "Reference" "#PWR0167" (id 0) (at 304.8 99.06 0)
       (effects (font (size 1.27 1.27)) hide)
     )
@@
   (symbol (lib_id "Device:L") (at 300.99 85.09 90) (unit 1)
     (in_bom yes) (on_board yes)
-    (property "Reference" "L?" (id 0) (at 300.99 86.36 90))
+    (property "Reference" "L2" (id 0) (at 300.99 86.36 90))
     (property "Value" "100u" (id 1) (at 300.99 82.55 90))
-    (property "Footprint" "" (id 2) (at 300.99 85.09 0)
+    (property "Footprint" "Anyleaf_Shared:SMNR4020 inductor" (id 2) (at 300.99 85.09 0)
       (effects (font (size 1.27 1.27)) hide)
     )
@@
       (effects (font (size 1.27 1.27)) hide)
     )
+    (property "LCSC" "C467068" (id 4) (at 300.99 85.09 90)
+      (effects (font (size 1.27 1.27)) hide)
+    )
     (pin "1")
     (pin "2")
@@
   (symbol (lib_id "Device:L") (at 267.97 43.18 0) (unit 1)
     (in_bom yes) (on_board yes) (fields_autoplaced)
-    (property "Reference" "L?" (id 0) (at 269.24 41.9099 0)
+    (property "Reference" "L1" (id 0) (at 269.24 41.9099 0)
       (effects (font (size 1.27 1.27)) (justify left))
     )
@@
     (pin "2")
   )
-  (symbol (lib_id "Device:C") (at 304.8 88.9 180) (unit 1)
-    (in_bom yes) (on_board yes)
-    (property "Reference" "C?" (id 0) (at 308.61 92.71 0)
-      (effects (font (size 1.27 1.27)) (justify right))
-    )
-    (property "Value" "C" (id 1) (at 308.61 90.1699 0)
-      (effects (font (size 1.27 1.27)) (justify right))
-    )
-    (property "Footprint" "" (id 2) (at 303.8348 85.09 0)
-      (effects (font (size 1.27 1.27)) hide)
-    )
-    (property "Datasheet" "~" (id 3) (at 304.8 88.9 0)
-      (effects (font (size 1.27 1.27)) hide)
-    )
-    (pin "1")
-    (pin "2")
-  )
   (symbol (lib_id "power:GND") (at 189.23 68.58 180) (unit 1)
     (in_bom yes) (on_board yes) (fields_autoplaced)
@@
     (pin "2")
   )
+  (symbol (lib_id "Device:C") (at 304.8 88.9 180) (unit 1)
+    (in_bom yes) (on_board yes)
+    (property "Reference" "C27" (id 0) (at 308.61 90.17 0)
+      (effects (font (size 1.27 1.27)) (justify left))
+    )
+    (property "Value" "47u" (id 1) (at 308.61 86.36 0)
+      (effects (font (size 1.27 1.27)) (justify left))
+    )
+    (property "Footprint" "Capacitor_SMD:C_0805_2012Metric" (id 2) (at 303.8348 85.09 0)
+      (effects (font (size 1.27 1.27)) hide)
+    )
+    (property "Datasheet" "~" (id 3) (at 304.8 88.9 0)
+      (effects (font (size 1.27 1.27)) hide)
+    )
+    (property "LCSC" "C16780" (id 4) (at 304.8 88.9 0)
+      (effects (font (size 1.27 1.27)) hide)
+    )
+    (pin "1")
+    (pin "2")
+  )
   (symbol (lib_id "power:+5V") (at 248.92 217.17 270) (unit 1)
     (in_bom yes) (on_board yes)
@@
   (symbol (lib_id "pspice:C") (at 265.43 62.23 0) (unit 1)
     (in_bom yes) (on_board yes) (fields_autoplaced)
-    (property "Reference" "C?" (id 0) (at 270.51 60.9599 0)
+    (property "Reference" "C26" (id 0) (at 270.51 60.9599 0)
       (effects (font (size 1.27 1.27)) (justify left))
     )
@@
     )
     (path "/5de18b47-f909-4eba-b434-657233f02ae6"
-      (reference "#PWR?") (unit 1) (value "GND") (footprint "")
+      (reference "#PWR0167") (unit 1) (value "GND") (footprint "")
     )
     (path "/4392ec2f-3eec-47ea-978d-f1725d990b74"
@@
       (reference "C25") (unit 1) (value "47u") (footprint "Capacitor_SMD:C_0805_2012Metric")
     )
-    (path "/baa1529e-ff54-4822-ab55-618d38eeeb89"
-      (reference "C?") (unit 1) (value "C") (footprint "")
-    )
     (path "/fcbac178-c57e-4596-b406-1b3b370d52dd"
-      (reference "C?") (unit 1) (value "C") (footprint "")
+      (reference "C26") (unit 1) (value "C") (footprint "")
+    )
+    (path "/f52e9835-147d-4eea-ab24-2abbf0cd1a27"
+      (reference "C27") (unit 1) (value "47u") (footprint "Capacitor_SMD:C_0805_2012Metric")
     )
     (path "/d692f2c3-969c-4042-b75e-63666695d58e"
@@
       (reference "J34") (unit 1) (value "Conn_01x01_Female") (footprint "TestPoint:TestPoint_Pad_1.0x1.0mm")
     )
-    (path "/16b4b87f-1be5-4fc9-8f1a-2362162eb831"
-      (reference "J35") (unit 1) (value "Conn_01x01_Female") (footprint "TestPoint:TestPoint_Pad_1.5x1.5mm")
-    )
     (path "/ef457e66-80d8-418f-b12e-08b7de05040b"
       (reference "J36") (unit 1) (value "Conn_01x01_Female") (footprint "TestPoint:TestPoint_Pad_1.5x1.5mm")
@@
       (reference "J51") (unit 1) (value "Conn_01x01_Female") (footprint "TestPoint:TestPoint_Pad_1.0x1.0mm")
     )
-    (path "/74196f2d-f470-4b2c-b15a-14b7f2f793d4"
-      (reference "L?") (unit 1) (value "100u") (footprint "")
-    )
     (path "/85e09d1b-23ff-4622-8dab-a4ac959ac541"
-      (reference "L?") (unit 1) (value "L") (footprint "")
+      (reference "L1") (unit 1) (value "L") (footprint "")
+    )
+    (path "/74196f2d-f470-4b2c-b15a-14b7f2f793d4"
+      (reference "L2") (unit 1) (value "100u") (footprint "Anyleaf_Shared:SMNR4020 inductor")
     )
     (path "/8a2f7ecd-dafc-493a-896e-651204d2233a"

Commit message: more work on CRSF radio comms
Parts:
- removed C26: C, symbol pspice:C
- removed L1: L, symbol Device:L
- U2: Digikey_ST_alt (none) -> 497-19784-1-ND
Other:
- note added: "ST modules like ISM330DHCX iNEMO appears to be pin compatible. That model is currently in stock at Digikey"
Changed lines of the file:
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@@
     (effects (font (size 1.27 1.27)) (justify left bottom))
   )
+  (text "ST modules like ISM330DHCX iNEMO\nappears to be pin compatible. That\nmodel is currently in stock at Digikey\n"
+    (at 195.58 64.77 0)
+    (effects (font (size 1.27 1.27)) (justify left bottom))
+  )
   (text "\"No external load capacitors are needed\"" (at 198.12 179.07 0)
     (effects (font (size 1.27 1.27)) (justify left bottom))
@@
     (effects (font (size 1.27 1.27)) (justify left bottom))
   )
+  (label "CS_FLASH" (at 158.75 104.14 180)
+    (effects (font (size 1.27 1.27)) (justify right bottom))
+  )
   (label "MISO_2" (at 190.5 227.33 180)
     (effects (font (size 1.27 1.27)) (justify right bottom))
@@
       (effects (font (size 1.27 1.27)) hide)
     )
+    (property "Digikey_ST_alt" "497-19784-1-ND" (id 7) (at 205.74 83.82 0)
+      (effects (font (size 1.27 1.27)) hide)
+    )
     (pin "1")
     (pin "12")
@@
     (pin "1")
   )
-  (symbol (lib_id "Device:L") (at 267.97 43.18 0) (unit 1)
-    (in_bom yes) (on_board yes) (fields_autoplaced)
-    (property "Reference" "L1" (id 0) (at 269.24 41.9099 0)
-      (effects (font (size 1.27 1.27)) (justify left))
-    )
-    (property "Value" "L" (id 1) (at 269.24 44.4499 0)
-      (effects (font (size 1.27 1.27)) (justify left))
-    )
-    (property "Footprint" "" (id 2) (at 267.97 43.18 0)
-      (effects (font (size 1.27 1.27)) hide)
-    )
-    (property "Datasheet" "~" (id 3) (at 267.97 43.18 0)
-      (effects (font (size 1.27 1.27)) hide)
-    )
-    (pin "1")
-    (pin "2")
-  )
   (symbol (lib_id "Device:C") (at 217.17 125.73 0) (unit 1)
     (in_bom yes) (on_board yes)
@@
     (pin "1")
   )
-  (symbol (lib_id "pspice:C") (at 265.43 62.23 0) (unit 1)
-    (in_bom yes) (on_board yes) (fields_autoplaced)
-    (property "Reference" "C26" (id 0) (at 270.51 60.9599 0)
-      (effects (font (size 1.27 1.27)) (justify left))
-    )
-    (property "Value" "C" (id 1) (at 270.51 63.4999 0)
-      (effects (font (size 1.27 1.27)) (justify left))
-    )
-    (property "Footprint" "" (id 2) (at 265.43 62.23 0)
-      (effects (font (size 1.27 1.27)) hide)
-    )
-    (property "Datasheet" "~" (id 3) (at 265.43 62.23 0)
-      (effects (font (size 1.27 1.27)) hide)
-    )
-    (pin "1")
-    (pin "2")
-  )
   (symbol (lib_id "Device:C") (at 123.19 38.1 0) (unit 1)
     (in_bom yes) (on_board yes)
@@
       (reference "C25") (unit 1) (value "47u") (footprint "Capacitor_SMD:C_0805_2012Metric")
     )
-    (path "/fcbac178-c57e-4596-b406-1b3b370d52dd"
-      (reference "C26") (unit 1) (value "C") (footprint "")
-    )
     (path "/f52e9835-147d-4eea-ab24-2abbf0cd1a27"
       (reference "C27") (unit 1) (value "47u") (footprint "Capacitor_SMD:C_0805_2012Metric")
@@
       (reference "J51") (unit 1) (value "Conn_01x01_Female") (footprint "TestPoint:TestPoint_Pad_1.0x1.0mm")
     )
-    (path "/85e09d1b-23ff-4622-8dab-a4ac959ac541"
-      (reference "L1") (unit 1) (value "L") (footprint "")
-    )
     (path "/74196f2d-f470-4b2c-b15a-14b7f2f793d4"

Commit message: Updated pin assignments
Connections:
- net CS_IMU: no longer U1.22 (PB10)
- net UART2_RX: now also U1.11 (PA3)
- net UART3_TX: now also U1.22 (PB10)
- net M1: now reaches U1.8 (PA0)
- net M1: now also J19.3 (Pin_3), J8.1 (Pin_1)
- removed net M1_PWM: J19.3 (Pin_3), J8.1 (Pin_1), U1.11 (PA3)
- net M2_PWM renamed M2
- net M3_PWM renamed M3
- net M4_PWM renamed M4
Other:
- note added: "M1: Tim2 Ch1 M2: Tim2 Ch4 M3: Tim3 Ch3 M4: Tim3 Ch4"
Changed lines of the file:
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@@
     (effects (font (size 1.27 1.27)) (justify right bottom))
+  )
+  (text "M1: Tim2 Ch1\nM2: Tim2 Ch4\nM3: Tim3 Ch3\nM4: Tim3 Ch4"
+    (at 146.05 53.34 0)
+    (effects (font (size 1.27 1.27)) (justify left bottom))
   )
   (text "See the MAX7456 datasheet for info on choosing\nC_OUT and C_SAG capacitors. Larger cap values\nresult in lower distortion. (But may be bulkier)"
@@
     (effects (font (size 1.27 1.27)) (justify left bottom))
   )
-  (label "M3_PWM" (at 377.19 35.56 180)
+  (label "M3" (at 377.19 35.56 180)
     (effects (font (size 1.27 1.27)) (justify right bottom))
   )
@@
     (effects (font (size 1.27 1.27)) (justify left bottom))
   )
-  (label "M2_PWM" (at 113.03 104.14 180)
-    (effects (font (size 1.27 1.27)) (justify right bottom))
-  )
-  (label "M2_PWM" (at 342.9 48.26 180)
+  (label "M2" (at 113.03 104.14 180)
+    (effects (font (size 1.27 1.27)) (justify right bottom))
+  )
+  (label "M2" (at 342.9 48.26 180)
     (effects (font (size 1.27 1.27)) (justify right bottom))
   )
@@
     (effects (font (size 1.27 1.27)) (justify right bottom))
   )
-  (label "M3_PWM" (at 143.51 60.96 0)
+  (label "M3" (at 143.51 60.96 0)
     (effects (font (size 1.27 1.27)) (justify left bottom))
   )
@@
     (effects (font (size 1.27 1.27)) (justify right bottom))
   )
-  (label "M4_PWM" (at 377.19 30.48 180)
+  (label "M4" (at 377.19 30.48 180)
     (effects (font (size 1.27 1.27)) (justify right bottom))
   )
@@
     (effects (font (size 1.27 1.27)) (justify right bottom))
   )
-  (label "M3_PWM" (at 342.9 45.72 180)
+  (label "M3" (at 342.9 45.72 180)
     (effects (font (size 1.27 1.27)) (justify right bottom))
   )
@@
     (effects (font (size 1.27 1.27)) (justify right bottom))
   )
-  (label "M4_PWM" (at 342.9 43.18 180)
+  (label "M4" (at 342.9 43.18 180)
     (effects (font (size 1.27 1.27)) (justify right bottom))
   )
@@
     (effects (font (size 1.27 1.27)) (justify left bottom))
   )
-  (label "M1_PWM" (at 377.19 45.72 180)
+  (label "M1" (at 377.19 45.72 180)
     (effects (font (size 1.27 1.27)) (justify right bottom))
   )
@@
     (effects (font (size 1.27 1.27)) (justify left bottom))
   )
-  (label "UART1_TX" (at 147.32 116.84 0)
+  (label "UART2_RX" (at 113.03 86.36 180)
+    (effects (font (size 1.27 1.27)) (justify right bottom))
+  )
+  (label "UART3_TX" (at 143.51 86.36 0)
     (effects (font (size 1.27 1.27)) (justify left bottom))
   )
@@
     (effects (font (size 1.27 1.27)) (justify left bottom))
   )
-  (label "CS_FLASH" (at 158.75 104.14 180)
-    (effects (font (size 1.27 1.27)) (justify right bottom))
+  (label "CS_FLASH" (at 165.1 91.44 0)
+    (effects (font (size 1.27 1.27)) (justify left bottom))
   )
   (label "MISO_2" (at 190.5 227.33 180)
@@
     (effects (font (size 1.27 1.27)) (justify left bottom))
   )
-  (label "M1_PWM" (at 113.03 86.36 180)
-    (effects (font (size 1.27 1.27)) (justify right bottom))
+  (label "M1" (at 113.03 78.74 180)
+    (effects (font (size 1.27 1.27)) (justify right bottom))
+  )
+  (label "GPIO" (at 165.1 93.98 0)
+    (effects (font (size 1.27 1.27)) (justify left bottom))
   )
   (label "VID_OUT" (at 374.65 114.3 180)
@@
     (effects (font (size 1.27 1.27)) (justify right bottom))
   )
-  (label "M4_PWM" (at 143.51 63.5 0)
+  (label "M4" (at 143.51 63.5 0)
     (effects (font (size 1.27 1.27)) (justify left bottom))
   )
@@
     (effects (font (size 1.27 1.27)) (justify right bottom))
   )
-  (label "M2_PWM" (at 377.19 40.64 180)
+  (label "M2" (at 377.19 40.64 180)
     (effects (font (size 1.27 1.27)) (justify right bottom))
   )
@@
     (effects (font (size 1.27 1.27)) (justify right bottom))
   )
-  (label "M1_PWM" (at 342.9 50.8 180)
+  (label "M1" (at 342.9 50.8 180)
     (effects (font (size 1.27 1.27)) (justify right bottom))
   )
@@
     (effects (font (size 1.27 1.27)) (justify right bottom))
   )
-  (label "CS_IMU" (at 143.51 86.36 0)
-    (effects (font (size 1.27 1.27)) (justify left bottom))
-  )
+  (label "CS_IMU" (at 165.1 88.9 0)
+    (effects (font (size 1.27 1.27)) (justify left bottom))
+  )
