File: circuit/quadcopter.kicad_sch (KiCad schematic)
At the start: 111 parts, among them J1 Conn_01x01_Female, J10 Conn_01x01_Female, J11 Conn_01x01_Female, J12 Conn_01x01_Female, J13 Conn_01x01_Female, J14 Conn_01x01_Female, J15 Conn_01x01_Female, J16 Conn_01x01_Female, J17 Conn_01x01_Female, J18 USB_C_Receptacle_USB2.0, J19 Conn_01x08_Male, J2 Conn_01x01_Female, J20 Conn_01x04_Male, J21 Conn_01x01_Female, J22 Conn_01x01_Female, J23 Conn_01x01_Female, J24 Conn_01x01_Female, J25 Conn_01x01_Female, J26 Conn_01x01_Female, J27 Conn_01x01_Female, J28 Conn_01x01_Female, J29 Conn_01x01_Female, J3 Conn_01x01_Female, J30 Conn_01x01_Female, J31 Conn_01x01_Female, J32 Conn_01x01_Female, J33 Conn_01x01_Female, J34 Conn_01x01_Female, J36 Conn_01x01_Female, J37 Conn_01x01_Female, J38 Conn_01x01_Female, J39 Conn_01x01_Female, J4 Conn_01x01_Female, J40 Conn_01x01_Female, J41 Conn_01x01_Female, J42 Conn_01x01_Female, J43 Conn_01x01_Female, J44 Conn_01x01_Female, J45 Conn_01x01_Female, J46 Conn_01x01_Female, J47 Conn_01x01_Female, J48 Conn_01x01_Female, J49 Conn_01x01_Female, J5 Conn_01x01_Female, J50 Conn_01x01_Female, J51 Conn_01x01_Female, J6 Conn_01x01_Female, J7 Conn_01x01_Female, J8 Conn_01x01_Female, J9 Conn_01x01_Female, SW1 SW_DIP_x01, U1 STM32G431CBU6, U2 ICM-42605, U3 DPS310, U4 3V3, U5 5V, U6 AT7456E, U7 W25Q128JVS, Y1 16M, Y2 27M

Commit message: Started work on RF circuit
Parts:
- added R13: 10k, Resistor_SMD:R_0402_1005Metric, symbol Device:R
- added R14: 1.5k, Resistor_SMD:R_0402_1005Metric, symbol Device:R
- J50: footprint TestPoint:TestPoint_Pad_2.0x2.0mm -> TestPoint:TestPoint_Pad_1.0x1.0mm
- Y1: footprint Oscillator:Oscillator_SMD_EuroQuartz_XO32-4Pin_3.2x2.5mm -> Crystal:Crystal_SMD_2016-4Pin_2.0x1.6mm; LCSC C13738 -> C254300
Connections:
- net +BATT: now also R13.2
- net GND: now also R14.1
- net BATT_DIV: now reaches U1.19 (PB2)
- net BATT_DIV: now also R13.1, R14.2
Other:
- note added: "Consider smaller crystals"
- note added: "Voltage divider. This keeps a 6S cell at full charge (25.2v) below 3.3v"
Changed lines of the file:
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@@
   (junction (at 266.7 55.88) (diameter 0) (color 0 0 0 0)
   )
+  (junction (at 58.42 109.22) (diameter 0) (color 0 0 0 0)
+  )
   (no_connect (at 113.03 66.04))
   (no_connect (at 113.03 68.58))
@@
     (stroke (width 0) (type default) (color 0 0 0 0))
   )
+  (wire (pts (xy 55.88 109.22) (xy 58.42 109.22))
+    (stroke (width 0) (type default) (color 0 0 0 0))
+  )
   (wire (pts (xy 184.15 204.47) (xy 185.42 204.47))
     (stroke (width 0) (type default) (color 0 0 0 0))
@@
     (stroke (width 0) (type default) (color 0 0 0 0))
   )
+  (wire (pts (xy 58.42 109.22) (xy 60.96 109.22))
+    (stroke (width 0) (type default) (color 0 0 0 0))
+  )
   (wire (pts (xy 100.33 68.58) (xy 111.76 68.58))
     (stroke (width 0) (type default) (color 0 0 0 0))
@@
     (stroke (width 0) (type default) (color 0 0 0 0))
   )
+  (wire (pts (xy 58.42 109.22) (xy 58.42 115.57))
+    (stroke (width 0) (type default) (color 0 0 0 0))
+  )
   (wire (pts (xy 121.92 48.26) (xy 124.46 48.26))
     (stroke (width 0) (type default) (color 0 0 0 0))
@@
     (effects (font (size 1.27 1.27)) (justify right bottom))
   )
+  (text "Voltage divider. This keeps a 6S cell\nat full charge (25.2v) below 3.3v"
+    (at 44.45 102.87 0)
+    (effects (font (size 1.27 1.27)) (justify left bottom))
+  )
   (text "Battery cicrcuit that includes a\nLC lowpass filter, to reduce noise from\nthe ESC."
     (at 261.62 95.25 0)
@@
     (effects (font (size 1.27 1.27)) (justify left bottom))
   )
+  (text "Consider smaller crystals" (at 69.85 88.9 0)
+    (effects (font (size 1.27 1.27)) (justify left bottom))
+  )
   (text "ST modules like ISM330DHCX iNEMO\nappears to be pin compatible. That\nmodel is currently in stock at Digikey\n"
     (at 195.58 64.77 0)
@@
     (effects (font (size 1.27 1.27)) (justify right bottom))
   )
+  (label "CURRENT" (at 165.1 86.36 0)
+    (effects (font (size 1.27 1.27)) (justify left bottom))
+  )
   (label "MISO_3" (at 143.51 71.12 0)
     (effects (font (size 1.27 1.27)) (justify left bottom))
@@
     (effects (font (size 1.27 1.27)) (justify right bottom))
   )
+  (label "BATT_DIV" (at 143.51 66.04 0)
+    (effects (font (size 1.27 1.27)) (justify left bottom))
+  )
   (label "MISO_3" (at 325.12 262.89 180)
     (effects (font (size 1.27 1.27)) (justify right bottom))
@@
     (effects (font (size 1.27 1.27)) (justify left bottom))
   )
-  (label "CS_FLASH" (at 165.1 91.44 0)
+  (label "CS_FLASH" (at 165.1 101.6 0)
     (effects (font (size 1.27 1.27)) (justify left bottom))
   )
@@
     (effects (font (size 1.27 1.27)) (justify right bottom))
   )
-  (label "GPIO" (at 165.1 93.98 0)
+  (label "BATT_DIV" (at 58.42 115.57 0)
+    (effects (font (size 1.27 1.27)) (justify left bottom))
+  )
+  (label "GPIO" (at 165.1 104.14 0)
     (effects (font (size 1.27 1.27)) (justify left bottom))
   )
@@
     (effects (font (size 1.27 1.27)) (justify right bottom))
   )
-  (label "CS_IMU" (at 165.1 88.9 0)
+  (label "CS_IMU" (at 165.1 99.06 0)
     (effects (font (size 1.27 1.27)) (justify left bottom))
   )
@@
     )
   )
+  (symbol (lib_id "power:+BATT") (at 48.26 109.22 90) (unit 1)
+    (in_bom yes) (on_board yes)
+    (property "Reference" "#PWR0169" (id 0) (at 52.07 109.22 0)
+      (effects (font (size 1.27 1.27)) hide)
+    )
+    (property "Value" "+BATT" (id 1) (at 44.45 109.22 90)
+      (effects (font (size 1.27 1.27)) (justify left))
+    )
+    (property "Footprint" "" (id 2) (at 48.26 109.22 0)
+      (effects (font (size 1.27 1.27)) hide)
+    )
+    (property "Datasheet" "" (id 3) (at 48.26 109.22 0)
+      (effects (font (size 1.27 1.27)) hide)
+    )
+    (pin "1")
+  )
   (symbol (lib_id "power:+3.3V") (at 194.31 121.92 90) (unit 1)
     (in_bom yes) (on_board yes)
@@
     (pin "2")
   )
+  (symbol (lib_id "Device:R") (at 52.07 109.22 270) (unit 1)
+    (in_bom yes) (on_board yes)
+    (property "Reference" "R13" (id 0) (at 52.07 106.68 90))
+    (property "Value" "10k" (id 1) (at 55.88 106.68 90))
+    (property "Footprint" "Resistor_SMD:R_0402_1005Metric" (id 2) (at 52.07 107.442 90)
+      (effects (font (size 1.27 1.27)) hide)
+    )
+    (property "Datasheet" "~" (id 3) (at 52.07 109.22 0)
+      (effects (font (size 1.27 1.27)) hide)
+    )
+    (property "LCSC" "C25744" (id 4) (at 52.07 109.22 0)
+      (effects (font (size 1.27 1.27)) hide)
+    )
+    (pin "1")
+    (pin "2")
+  )
   (symbol (lib_id "Device:C") (at 182.88 72.39 0) (unit 1)
     (in_bom yes) (on_board yes)
@@
       (effects (font (size 1.27 1.27)) (justify left))
     )
-    (property "Footprint" "TestPoint:TestPoint_Pad_2.0x2.0mm" (id 2) (at 330.2 223.52 0)
+    (property "Footprint" "TestPoint:TestPoint_Pad_1.0x1.0mm" (id 2) (at 330.2 223.52 0)
       (effects (font (size 1.27 1.27)) hide)
     )
@@
     (property "Reference" "Y1" (id 0) (at 102.87 67.31 90))
     (property "Value" "16M" (id 1) (at 97.79 67.31 90))
-    (property "Footprint" "Oscillator:Oscillator_SMD_EuroQuartz_XO32-4Pin_3.2x2.5mm" (id 2) (at 100.33 72.39 0)
+    (property "Footprint" "Crystal:Crystal_SMD_2016-4Pin_2.0x1.6mm" (id 2) (at 100.33 72.39 0)
       (effects (font (size 1.27 1.27)) hide)
     )
-    (property "Datasheet" "https://datasheet.lcsc.com/lcsc/2103291133_Yangxing-Tech-X322516MLB4SI_C13738.pdf" (id 3) (at 100.33 72.39 0)
+    (property "Datasheet" "https://datasheet.lcsc.com/lcsc/1912111437_HELE-Harmony-Elec-X2C016000B81H-R_C254300.pdf" (id 3) (at 100.33 72.39 0)
       (effects (font (size 1.27 1.27)) hide)
     )
-    (property "LCSC" "C13738" (id 4) (at 100.33 72.39 0)
+    (property "LCSC" "C254300" (id 4) (at 100.33 72.39 0)
       (effects (font (size 1.27 1.27)) hide)
     )
@@
     (pin "1")
   )
+  (symbol (lib_id "Device:R") (at 64.77 109.22 270) (unit 1)
+    (in_bom yes) (on_board yes)
+    (property "Reference" "R14" (id 0) (at 64.77 106.68 90))
+    (property "Value" "1.5k" (id 1) (at 68.58 106.68 90))
+    (property "Footprint" "Resistor_SMD:R_0402_1005Metric" (id 2) (at 64.77 107.442 90)
+      (effects (font (size 1.27 1.27)) hide)
+    )
+    (property "Datasheet" "~" (id 3) (at 64.77 109.22 0)
+      (effects (font (size 1.27 1.27)) hide)
+    )
+    (property "LCSC" "C25867" (id 4) (at 64.77 109.22 0)
+      (effects (font (size 1.27 1.27)) hide)
+    )
+    (pin "1")
+    (pin "2")
+  )
   (symbol (lib_id "Connector:Conn_01x01_Female") (at 330.2 218.44 0) (unit 1)
     (in_bom yes) (on_board yes) (fields_autoplaced)
@@
     (pin "1")
   )
+  (symbol (lib_id "power:GND") (at 68.58 109.22 90) (unit 1)
+    (in_bom yes) (on_board yes)
+    (property "Reference" "#PWR0168" (id 0) (at 74.93 109.22 0)
+      (effects (font (size 1.27 1.27)) hide)
+    )
+    (property "Value" "GND" (id 1) (at 71.8312 109.093 90)
+      (effects (font (size 1.27 1.27)) (justify right))
+    )
+    (property "Footprint" "" (id 2) (at 68.58 109.22 0)
+      (effects (font (size 1.27 1.27)) hide)
+    )
+    (property "Datasheet" "" (id 3) (at 68.58 109.22 0)
+      (effects (font (size 1.27 1.27)) hide)
+    )
+    (pin "1")
+  )
   (symbol (lib_id "Device:R") (at 229.87 210.82 180) (unit 1)
     (in_bom yes) (on_board yes)
@@
       (reference "#PWR0167") (unit 1) (value "GND") (footprint "")
     )
+    (path "/76f68b18-fc7d-4be2-b12c-66e2770ae749"
+      (reference "#PWR0168") (unit 1) (value "GND") (footprint "")
+    )
+    (path "/3a0746df-74de-4d9e-bc61-8916d85d8abe"
+      (reference "#PWR0169") (unit 1) (value "+BATT") (footprint "")
+    )
     (path "/4392ec2f-3eec-47ea-978d-f1725d990b74"
       (reference "C1") (unit 1) (value "2.2u") (footprint "Capacitor_SMD:C_0402_1005Metric")
@@
     )
     (path "/539aff64-906a-4c96-9d13-3f8f7fef9048"
-      (reference "J50") (unit 1) (value "Conn_01x01_Female") (footprint "TestPoint:TestPoint_Pad_2.0x2.0mm")
+      (reference "J50") (unit 1) (value "Conn_01x01_Female") (footprint "TestPoint:TestPoint_Pad_1.0x1.0mm")
     )
     (path "/b6907dd4-a67f-45c4-ba83-8e8c1e0e318c"
@@
       (reference "R12") (unit 1) (value "22") (footprint "Resistor_SMD:R_0402_1005Metric")
     )
+    (path "/427ea469-a00c-48a4-8283-a7d9e027923d"
+      (reference "R13") (unit 1) (value "10k") (footprint "Resistor_SMD:R_0402_1005Metric")
+    )
+    (path "/667f12d7-16dd-4278-bb5b-b991203c0138"
+      (reference "R14") (unit 1) (value "1.5k") (footprint "Resistor_SMD:R_0402_1005Metric")
+    )
     (path "/2215b67b-b7c5-48e7-ada2-5ba365cf8893"
       (reference "SW1") (unit 1) (value "SW_DIP_x01") (footprint "Anyleaf_Shared:SW-SMD-2_3.6x6.0x8.0")
@@
     )
     (path "/5e9abcd9-0fc4-4926-b01a-9cedb724738c"
-      (reference "Y1") (unit 1) (value "16M") (footprint "Oscillator:Oscillator_SMD_EuroQuartz_XO32-4Pin_3.2x2.5mm")
+      (reference "Y1") (unit 1) (value "16M") (footprint "Crystal:Crystal_SMD_2016-4Pin_2.0x1.6mm")
     )
     (path "/efb1f23e-5469-49d3-92f6-7fe3219fa856"

Commit message: Lots of work on schematic, and BF cfg
Parts:
- removed J11: Conn_01x01_Female, TestPoint:TestPoint_Pad_1.5x1.5mm, symbol Connector:Conn_01x01_Female
- removed J14, J5, J51, J6: Conn_01x01_Female, TestPoint:TestPoint_Pad_1.0x1.0mm, symbol Connector:Conn_01x01_Female
- removed J20: Conn_01x04_Male, Connector_JST:JST_SH_SM04B-SRSS-TB_1x04-1MP_P1.00mm_Horizontal, symbol Connector:Conn_01x04_Male
- added AE1: Antenna, Connector_Coaxial:U.FL_Molex_MCRF_73412-0110_Vertical, symbol Device:Antenna
- added C26, C28, C29, C30: 100n, Capacitor_SMD:C_0402_1005Metric, symbol Device:C
- added J5: Conn_01x07_Male, Connector_JST:JST_SH_BM07B-SRSS-TB_1x07-1MP_P1.00mm_Vertical, symbol Connector:Conn_01x07_Male
- added R15, R16: 10k, Resistor_SMD:R_0402_1005Metric, symbol Device:R
- added R17, R18: 1.5k, Resistor_SMD:R_0402_1005Metric, symbol Device:R
- added U8: SX1281, Package_DFN_QFN:QFN-24-1EP_4x4mm_P0.5mm_EP2.6x2.6mm, symbol Anyleaf_Shared:SX1281
Connections:
- net +3V3: now also C26.2, C28.2, C29.2, C30.2, U8.1 (VR_PA), U8.11 (VBAT_IO), U8.15 (VBAT), U8.2 (VDD_IN), U8.6 (XTB)
- net +5V: now also J26.1 (Pin_1), J5.2 (Pin_2)
- net +BATT: now also J5.5 (Pin_5); no longer J26.1 (Pin_1)
- net CS_FLASH: now also U1.2 (PC13)
- net CS_IMU: now also U1.25 (PB12)
- net CURRENT: now also R16.2
- net ESC_TELE: no longer J22.1 (Pin_1)
- net GND: now also C26.1, C28.1, C29.1, C30.1, J5.3 (Pin_3), J5.4 (Pin_4), R17.1, R18.1, U8.13 (GND), U8.15 (VBAT), U8.20 (GND), U8.21 (GND), U8.22 (GND), U8.23 (GND), U8.24 (GND), U8.25 (EP_GND), U8.5 (GND)
- net MISO_3: now also U8.16 (MISO_TX)
- net MOSI_3: now also U8.17 (MOSI_RX)
- net RSSI: now also J5.7 (Pin_7), R15.2
- net SCK_3: now also U8.18 (SCK_RTSN)
- net UART3_RX: now also J22.1 (Pin_1)
- net VID_IN: now also J5.1 (Pin_1)
- net VID_OUT: now also J5.6 (Pin_6)
- net CS_ELRS: now reaches U1.4 (PC15-OSC32_OUT)
- net CS_ELRS: now also U8.19 (NSS_CTS)
- new net CUR_DIV: R16.1, R18.2
- new net RSSI_DIV: R15.1, R17.2
- no-connect marks 5 -> 3
Other:
- note added: "ELRS receiver"
- note added: "Header to connect to Rx, and VTX."
- note added: "IPEX MHF antenna port?"
- note added: "Telemetry"
- note added: "todo: What resistor vls for RSSI adn cur?"
- moved on the sheet: J12, J25, J26

Commit message: More work routing
Parts:
- added J11: Conn_01x03_Male, Connector_JST:JST_SH_BM03B-SRSS-TB_1x03-1MP_P1.00mm_Vertical, symbol Connector:Conn_01x03_Male
- added J6: Conn_01x04_Male, Connector_JST:JST_SH_BM04B-SRSS-TB_1x04-1MP_P1.00mm_Vertical, symbol Connector:Conn_01x04_Male
Connections:
- net +3V3: now also U8.3 (NRESET); no longer U8.6 (XTB)
- net +5V: now also J11.2 (Pin_2)
- net +BATT: now also J6.2 (Pin_2)
- net GND: now also J11.1 (Pin_1), J6.1 (Pin_1); no longer U8.22 (GND)
- net MISO_2: now also U8.16 (MISO_TX)
- net MISO_3: no longer U8.16 (MISO_TX)
- net MOSI_2: now also U8.17 (MOSI_RX)
- net MOSI_3: no longer U8.17 (MOSI_RX)
- net RSSI: now also J6.4 (Pin_4)
- net SCK_2: now also U8.18 (SCK_RTSN)
- net SCK_3: no longer U8.18 (SCK_RTSN)
- net VID_IN: now also J11.3 (Pin_3)
- net VID_OUT: now also J6.3 (Pin_3)
- net at AE1.1 (A): now also U8.22 (RFIO)
- no-connect marks 3 -> 10
Other:
- moved on the sheet: AE1, U8

Commit message: Translated much of the BF ELRS code
Connections:
- net MISO_2: no longer U8.16 (MISO_TX)
- net MISO_3: now also U8.16 (MISO_TX)
- net MOSI_2: no longer U8.17 (MOSI_RX)
- net MOSI_3: now also U8.17 (MOSI_RX)
- net SCK_2: no longer U8.18 (SCK_RTSN)
- net SCK_3: now also U8.18 (SCK_RTSN)
- net ELRS_BUSY: now reaches U8.7 (BUSY)
Changed lines of the file:
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@@
     (effects (font (size 1.27 1.27)) (justify left bottom))
   )
-  (label "MOSI_2" (at 78.74 303.53 0)
+  (label "MOSI_3" (at 78.74 303.53 0)
     (effects (font (size 1.27 1.27)) (justify left bottom))
   )
@@
     (effects (font (size 1.27 1.27)) (justify right bottom))
   )
+  (label "ELRS_BUSY" (at 48.26 297.18 180)
+    (effects (font (size 1.27 1.27)) (justify right bottom))
+  )
   (label "SCL2" (at 194.31 116.84 180)
     (effects (font (size 1.27 1.27)) (justify right bottom))
@@
     (effects (font (size 1.27 1.27)) (justify left bottom))
   )
-  (label "SCK_2" (at 78.74 300.99 0)
+  (label "SCK_3" (at 78.74 300.99 0)
     (effects (font (size 1.27 1.27)) (justify left bottom))
   )
@@
     (effects (font (size 1.27 1.27)) (justify right bottom))
   )
+  (label "ELRS_BUSY" (at 165.1 104.14 0)
+    (effects (font (size 1.27 1.27)) (justify left bottom))
+  )
   (label "UART4_RX" (at 375.92 210.82 180)
     (effects (font (size 1.27 1.27)) (justify right bottom))
@@
     (effects (font (size 1.27 1.27)) (justify left bottom))
   )
-  (label "MISO_2" (at 78.74 306.07 0)
-    (effects (font (size 1.27 1.27)) (justify left bottom))
-  )
+  (label "MISO_3" (at 78.74 306.07 0)
+    (effects (font (size 1.27 1.27)) (justify left bottom))
+  )
