File: circuit/quadcopter.kicad_sch (KiCad schematic)
At the start: 117 parts, among them J1 Conn_01x01_Female, J10 Conn_01x01_Female, J12 Conn_01x01_Female, J13 Conn_01x01_Female, J15 Conn_01x01_Female, J16 Conn_01x01_Female, J17 Conn_01x01_Female, J18 USB_C_Receptacle_USB2.0, J19 Conn_01x08_Male, J2 Conn_01x01_Female, J21 Conn_01x01_Female, J22 Conn_01x01_Female, J23 Conn_01x01_Female, J24 Conn_01x01_Female, J25 Conn_01x01_Female, J26 Conn_01x01_Female, J28 Conn_01x01_Female, J29 Conn_01x01_Female, J30 Conn_01x01_Female, J31 Conn_01x01_Female, J32 Conn_01x01_Female, J33 Conn_01x01_Female, J34 Conn_01x01_Female, J36 Conn_01x01_Female, J37 Conn_01x01_Female, J38 Conn_01x01_Female, J39 Conn_01x01_Female, J40 Conn_01x01_Female, J41 Conn_01x01_Female, J42 Conn_01x01_Female, J43 Conn_01x01_Female, J44 Conn_01x01_Female, J45 Conn_01x01_Female, J46 Conn_01x01_Female, J47 Conn_01x01_Female, J48 Conn_01x01_Female, J49 Conn_01x01_Female, J5 Conn_Coaxial, J50 Conn_01x01_Female, J6 Conn_01x06_Male, J7 Conn_01x01_Female, J8 Conn_01x01_Female, J9 Conn_01x01_Female, SW1 SW_DIP_x01, U1 STM32G431CBU6, U2 ICM-42605, U3 DPS310, U4 3V3, U5 5V, U6 AT7456E, U7 W25Q128JVS, U8 SX1281, Y1 16M, Y2 27M

Commit message: Added buzzer supporting circuitry. Minor code changes
Parts:
- removed J36: Conn_01x01_Female, TestPoint:TestPoint_Pad_1.5x1.5mm, symbol Connector:Conn_01x01_Female
- added Q1: AO3400A, Package_TO_SOT_SMD:SOT-23, symbol Anyleaf_Shared:AO3400A
- added R15: 10k, Resistor_SMD:R_0402_1005Metric, symbol Device:R
- H9: footprint Anyleaf_Shared:Mouse bites_5mm -> Anyleaf_Shared:Mouse bites_7mm
Connections:
- net +5V: now also J37.1 (Pin_1)
- net GND: now also Q1.2 (S), R15.1; no longer J37.1 (Pin_1)
- net ELRS_DIO: now reaches U8.8 (DIO1)
- net ELRS_DIO: now also U1.9 (PA1)
- net BUZZER+ renamed BUZZER-
- net BUZZER-: now also Q1.3 (D)
- net ELRS_RST: no longer names the net of U8.3 (NRESET)
- net ELRS_RST: no longer U1.9 (PA1)
- new net BUZZER_PWM: Q1.1 (G), R15.2
- no-connect marks 13 -> 12
Other:
- note added: "Example full buzzer circuit. Not on BOM!"
- note added: "How to wire buzzer pins?"
- note added: "ST modules like ISM330DHCX iNEMO appears to be pin compatible. That model is currently in stock at Digikey. Also compatible with BMI270. If using that, check pins 2,3,10,11 acceptable values"
- note added: "This transisor switch circuit allows 5V across the, using the 3V3 PWM signal."
- note added: "We currently use I2C for the DPS310 barometer. Connecting CSB high selects this."
- note added: "What voltage divider on current sense?"
- note added: "todo: Do we need rst?"
- note added: "todo: Xtal connection on SX1280? If not, does/can it get clock from MCU?"
- note removed: "IPEX MHF antenna port?"
- note removed: "ST modules like ISM330DHCX iNEMO appears to be pin compatible. That model is currently in stock at Digikey. Also compatible with __"
- note removed: "We currently use I2C for the DPS310 barometer. Connected CSB high selects this."
- moved on the sheet: J31, J37

Commit message: More work on PCB, and ELRS code
Parts:
- added J3: Conn_01x01_Female, TestPoint:TestPoint_Pad_1.5x1.5mm, symbol Connector:Conn_01x01_Female
- C14: value 10u -> 10uF 50V; footprint Capacitor_SMD:C_0402_1005Metric -> Capacitor_SMD:C_0805_2012Metric; LCSC C15525 -> C440198
- C15: value 10u -> 10uF 10V; footprint Capacitor_SMD:C_0402_1005Metric -> Capacitor_SMD:C_0603_1608Metric; LCSC C15525 -> C19702
- C27: value 47u -> 22u 35v; LCSC C16780 -> C338080
- C7: value 1u -> 1u 50V; footprint Capacitor_SMD:C_0402_1005Metric -> Capacitor_SMD:C_0603_1608Metric; LCSC C52923 -> C15849
- D1, D2: value MBR0530 -> 40v 1A B5819WS; footprint Diode_SMD:D_SOD-123 -> Diode_SMD:D_SOD-323; LCSC C82046 -> C22624
- Q1, R15: now left out of the parts list
Connections:
- net BUZZER_PWM: now also J31.1 (Pin_1), U1.29 (PC6)
- net GND: now also J3.1 (Pin_1)
- removed net BUZZER-: J31.1 (Pin_1), Q1.3 (D), U1.29 (PC6)
- new net BUZZER: Q1.3 (D)
- no-connect marks 12 -> 13
Other:
- note added: "TODO: Cap on batt is far too low v!! on 5v, should bve higher too."
- note added: "todo: Check max v on inductor"
- moved on the sheet: J31, J37

Commit message: More work on tweaking PCB layout
Parts:
- added C31: 100u, Capacitor_SMD:C_0805_2012Metric, symbol Device:C
- added L1: 10u, Inductor_SMD:L_0603_1608Metric, symbol Device:L
- F1: now left out of the parts list
- U5: value 5V -> 5V out, 30V max
Connections:
- net +3V3: now also L1.1; no longer C1.2, C3.2, C4.1, U2.5 (VDDIO), U2.8 (VDD)
- net GND: now also C31.1
- net at F1.1: no longer D1.2 (A)
- net at J18.A4 (VBUS), J18.A9 (VBUS), J18.B4 (VBUS)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: now also D1.2 (A); no longer F1.2
- new net: C1.2, C3.2, C31.2, C4.1, L1.2, U2.5 (VDDIO), U2.8 (VDD)
Other:
- note added: "LDO voltage too low. Try again!"
- note added: "Note: Removed fuse on USB to save space"
- note added: "Note: This cap is expensive, but is a smaller footprint than others of this cap"
- note added: "Separate and filter IMU power supply from the rest of the 3v3 line. LC filter."
- note removed: "TODO: Cap on batt is far too low v!! on 5v, should bve higher too."
- moved on the sheet: C1, C2, C3, C4, C5, F1, U2, U3

Commit message: Basic layout for OSD-less MCU in progress
Parts:
- removed C19, C20, C21, C22: 100n, Capacitor_SMD:C_0402_1005Metric, symbol Device:C
- removed C24, C25: 47u, Capacitor_SMD:C_0805_2012Metric, symbol Device:C
- removed J12: Conn_01x01_Female, TestPoint:TestPoint_Pad_1.5x1.5mm, symbol Connector:Conn_01x01_Female
- removed R10, R11: 75, Resistor_SMD:R_0402_1005Metric, symbol Device:R
- removed R7, R8, R9: 1k, Resistor_SMD:R_0402_1005Metric, symbol Device:R
- removed U6: AT7456E, Package_SO:TSSOP-28_4.4x9.7mm_P0.65mm, symbol Anyleaf_Shared:AT7456E
- removed Y2: 27M, Oscillator:Oscillator_SMD_EuroQuartz_XO32-4Pin_3.2x2.5mm, symbol Device:Crystal_GND24
- F1: now in the parts list
- J50: footprint TestPoint:TestPoint_Pad_1.0x1.0mm -> TestPoint:TestPoint_Pad_2.0x2.0mm
- R6: now left out of the parts list
- U7: value W25Q128JVS -> W25Q80DVUXIE TR; Digikey (none) -> W25Q80DVUXIETR-ND
Connections:
- net +3V3: now also SW1.2; no longer R6.2
- net MISO_2: now also U7.2 (DO(IO1))
- net MISO_3: no longer U7.2 (DO(IO1))
- net MOSI_2: now also U7.5 (DI(IO0))
- net MOSI_3: no longer U7.5 (DI(IO0))
- net SCK_2: now also U7.6 (CLK)
- net SCK_3: no longer U7.6 (CLK)
- net at R6.1: no longer SW1.2
- net at F1.1: now also D1.2 (A)
- net at F1.2: now also J18.A4 (VBUS), J18.A9 (VBUS), J18.B4 (VBUS), J18.B9 (VBUS)
- no-connect marks 13 -> 11
Other:
- note added: "This resistor pulling boot0 high is removed; probably not required, although present on STM32 dev boards"
- note added: "todo: Higher capacity flash"
- note added: "todo: Temporarily removed this IMU pwr filtering due to size"
- note added: "todo: Xtal connection on SX1280! If not, does/can it get clock from MCU?"
- note removed: ""No external load capacitors are needed""
- note removed: "On screen display (Analog)"
- note removed: "See the MAX7456 datasheet for info on choosing C_OUT and C_SAG capacitors. Larger cap values result in lower distortion. (But may be bulkier)"
- note removed: "todo: Check voltage req of C_x caps. Currently at 6v. Use 1206 for 10v"
- note removed: "todo: Xtal connection on SX1280? If not, does/can it get clock from MCU?"
- moved on the sheet: C31, F1, L1, R6

Commit message: More work on PCB
Parts:
- removed J38, J39: Conn_01x01_Female, TestPoint:TestPoint_Pad_2.0x2.0mm, symbol Connector:Conn_01x01_Female
- added J4: Conn_01x01_Female, TestPoint:TestPoint_Pad_1.5x1.5mm, symbol Connector:Conn_01x01_Female
- L1: value 10u -> 100u 450mA; footprint Inductor_SMD:L_0603_1608Metric -> Anyleaf_Shared:SMNR4020 inductor; LCSC C1035 -> C467068
- L2: value 100u -> 100u 450mA
Connections:
- net VID_IN is gone; now on net +BATT: J6.6 (Pin_6)
- net +5V: no longer J26.1 (Pin_1), J6.5 (Pin_5)
- net +BATT: now also J25.1 (Pin_1); no longer J29.1 (Pin_1), J6.2 (Pin_2)
- net BATT_DIV: now also U1.12 (PA4); no longer U1.16 (PC4)
- net GND: now also J26.1 (Pin_1), J29.1 (Pin_1), J6.2 (Pin_2), J6.5 (Pin_5); no longer J25.1 (Pin_1), J28.1 (Pin_1), J6.1 (Pin_1), J6.4 (Pin_4)
- net IMU_INTERRUPT: now also U1.16 (PC4); no longer U1.12 (PA4)
- net UART1_RX: now also J28.1 (Pin_1), J6.3 (Pin_3)
- net UART1_TX: now also J13.1 (Pin_1), J6.4 (Pin_4)
- net UART2_RX: now also J6.1 (Pin_1), J4.1 (Pin_1)
- net VID_OUT: no longer J13.1 (Pin_1), J6.3 (Pin_3)
- net IMU_pwr: now reaches C1.2, C3.2, C31.2, C4.1, L1.2, U2.5 (VDDIO), U2.8 (VDD)
Other:
- note added: "(HDL / SBUS)"
- note added: "7-26V for both HD-zero and DJI, so can't use with 8S battery!"
- note added: "Digital camera/Vtx pins and pads. DJI layout. Hd-zero layout is GND, Pwr, Rx, Tx, (sometimes Smart Audio and/or SBUS?)"
- note removed: "Analog camera"
- note removed: "Analog vid transmitter"
- note removed: "Header to connect to Rx, and VTX."
- note removed: "LDO voltage too low. Try again!"
- note removed: "Note: This cap is expensive, but is a smaller footprint than others of this cap"
- moved on the sheet: C14, C15, C27, C31, D2, J13, J19, J25, J26, J28, J29, J6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

Commit message: Added filtering /decoupling circuitry to LoRa chip. More work on board routing
Parts:
- removed C26: 100n, Capacitor_SMD:C_0402_1005Metric, symbol Device:C
- added C19: 10n, Capacitor_SMD:C_0402_1005Metric, symbol Device:C
- added C20: .8p (actual: 1pF), Capacitor_SMD:C_0402_1005Metric, symbol Device:C
- added C21, C24: 1.2p, Capacitor_SMD:C_0402_1005Metric, symbol Device:C
- added C22: 0.5p, Capacitor_SMD:C_0402_1005Metric, symbol Device:C
- added C25: 100p, Capacitor_SMD:C_0402_1005Metric, symbol Device:C
- added C?: 470n, 10V, Capacitor_SMD:C_0402_1005Metric, symbol Device:C
- added L3: 15u, Inductor_SMD:L_0805_2012Metric, symbol Device:L
- added L4: 3n, Inductor_SMD:L_0402_1005Metric, symbol Device:L
- added L5: 2.5n (3n actual), Inductor_SMD:L_0402_1005Metric, symbol Device:L
- added Y2: 52Mhz, Crystal:Crystal_SMD_2016-4Pin_2.0x1.6mm, symbol Device:Crystal_GND24
- C28: value 100n -> 10n; LCSC C1525 -> C15195
Connections:
- net +3V3: no longer C28.2, C29.2, C30.2, U8.1 (VR_PA), U8.11 (VBAT_IO), U8.15 (VBAT), U8.2 (VDD_IN)
- net GND: now also C19.1, C20.2, C21.2, C24.2, C?.2, Y2.2, Y2.4
- net UART2_RX: no longer J4.1 (Pin_1)
- net UART2_TX: now also J4.1 (Pin_1)
- net at U8.22 (RFIO): now also C20.1, L4.1; no longer J5.1 (In)
- net at U8.4 (XTA): now also Y2.1
- net at U8.6 (XTB): now also Y2.3
- new net: C21.1, C22.1, L4.2, L5.1
- new net: C28.2, C?.1, L3.1, U8.2 (VDD_IN)
- new net: C22.2, C24.1, C25.1, L5.2
- new net: C19.2, U8.1 (VR_PA)
- new net: C25.2, J5.1 (In)
- no-connect marks 11 -> 9
Other:
- note added: "Note: Voltage range of CADDX vista DJI: 7.4 - 26.4V HDzero: Racev2: 7-26V Hdzero freestyle: 7-17V max (4S!)"
- note added: "Reference SX1280 Datsheet, section 15.1: Reference Design"
- note removed: "ESC (iflight-layout header)"
- note removed: "todo: Do we need rst?"
- note removed: "todo: Temporarily removed this IMU pwr filtering due to size"
- note removed: "todo: Xtal connection on SX1280! If not, does/can it get clock from MCU?"
- moved on the sheet: C2, C5, J5, U3
