File: circuit_rf/circuit_rf.kicad_pcb (KiCad board)
At the start: 4 copper layers, 37.7 x 37.7 mm, 21 parts, among them J18 USB_C_Receptacle_USB2.0, U8 ESP32-C3, U9 SX1279, Y1 16M

Commit message: Lots of work on schematic, and BF cfg
Parts:
- removed U8: ESP32-C3, Package_DFN_QFN:QFN-32-1EP_5x5mm_P0.5mm_EP3.7x3.7mm
- added BZ1: Buzzer, Anyleaf_Shared:Buzzer_MLT-7525, F.Cu at (174.0, 107.2)
- added C1: 100n, Capacitor_SMD:C_0402_1005Metric, F.Cu at (132.0, 83.8)
- added C10: 100n, Capacitor_SMD:C_0402_1005Metric, F.Cu at (198.9, 92.2)
- added C11: 100n, Capacitor_SMD:C_0402_1005Metric, F.Cu at (126.8, 103.0)
- added C2: 100n, Capacitor_SMD:C_0402_1005Metric, F.Cu at (132.0, 86.5)
- added C3: 100n, Capacitor_SMD:C_0402_1005Metric, F.Cu at (137.0, 92.2)
- added C4: 100n, Capacitor_SMD:C_0402_1005Metric, F.Cu at (140.2, 82.8)
- added C5: 100n, Capacitor_SMD:C_0402_1005Metric, F.Cu at (142.2, 90.5)
- added C6: 100n, Capacitor_SMD:C_0402_1005Metric, F.Cu at (201.8, 92.2)
- added C7: 100n, Capacitor_SMD:C_0402_1005Metric, F.Cu at (196.0, 92.2)
- added C8: 100n, Capacitor_SMD:C_0402_1005Metric, F.Cu at (196.0, 94.2)
- added C9: 100n, Capacitor_SMD:C_0402_1005Metric, F.Cu at (198.9, 94.2)
- added Q1: AO3400A, Package_TO_SOT_SMD:SOT-23, F.Cu at (181.6, 105.2)
- added R1: 10k, Resistor_SMD:R_0402_1005Metric, F.Cu at (180.6, 108.4)
- added U1: ESP32-PICO-D4, Package_DFN_QFN:QFN-48-1EP_7x7mm_P0.5mm_EP5.3x5.3mm, F.Cu at (137.0, 87.5)
- added Ue: ESP32-WROOM-32U, RF_Module:ESP32-WROOM-32U, F.Cu at (97.8, 85.0)
Connections:
- U9 pad 14: unconnected-(U9-Pad14) -> +3V3
- U9 pad 15: Net-(U9-Pad15) -> GND
- U9 pad 2: unconnected-(U9-Pad2) -> +3V3
- U9 pad 23: Net-(U9-Pad15) -> GND
- U9 pad 24: unconnected-(U9-Pad24) -> +3V3
- U9 pad 26: Net-(U9-Pad15) -> GND
- U9 pad 29: Net-(U9-Pad15) -> GND
- U9 pad 3: unconnected-(U9-Pad3) -> +3V3
- U9 pad 4: unconnected-(U9-Pad4) -> +3V3
Routing:
- net GND: vias 0 -> 5
